Commit message: feat(urdf): resize mount plate and offset UR10e to avoid column collision

File: src/prismatic_7dof_sim/model/prismatic_ur10e.urdf.xacro (robot description, xacro)
@@ -105,5 +105,5 @@
       <origin xyz="0 0 ${mount_plate_height / 2.0}" rpy="0 0 0"/>
       <geometry>
-        <box size="0.35 0.35 ${mount_plate_height}"/>
+        <box size="0.75 0.35 ${mount_plate_height}"/>
       </geometry>
       <material name="lift_light"/>
@@ -112,5 +112,5 @@
       <origin xyz="0 0 ${mount_plate_height / 2.0}" rpy="0 0 0"/>
       <geometry>
-        <box size="0.35 0.35 ${mount_plate_height}"/>
+        <box size="0.75 0.35 ${mount_plate_height}"/>
       </geometry>
     </collision>
@@ -122,7 +122,7 @@
         ixy="0.0"
         ixz="0.0"
-        iyy="${mount_plate_mass * (0.35 * 0.35 + mount_plate_height * mount_plate_height) / 12.0}"
+        iyy="${mount_plate_mass * (0.75 * 0.75 + mount_plate_height * mount_plate_height) / 12.0}"
         iyz="0.0"
-        izz="${mount_plate_mass * (0.35 * 0.35 + 0.35 * 0.35) / 12.0}"/>
+        izz="${mount_plate_mass * (0.75 * 0.75 + 0.35 * 0.35) / 12.0}"/>
     </inertial>
   </link>
@@ -139,7 +139,6 @@
     kinematics_parameters_file="$(find ur_description)/config/$(arg ur_type)/default_kinematics.yaml"
     physical_parameters_file="$(find ur_description)/config/$(arg ur_type)/physical_parameters.yaml"
-    visual_parameters_file="$(find ur_description)/config/$(arg ur_type)/visual_parameters.yaml"
-    generate_ros2_control_tag="false">
-    <origin xyz="0 0 ${mount_plate_height}" rpy="0 0 0"/>
+    visual_parameters_file="$(find ur_description)/config/$(arg ur_type)/visual_parameters.yaml">
+    <origin xyz="-0.25 0 ${mount_plate_height}" rpy="0 0 0"/>
   </xacro:ur_robot>
   <gazebo>
